File: C64 Joystick Switcher.sch (KiCad schematic (older format))
At the start: 30 parts, among them J1 Port 1, J2 Port 2, J3 Joystick, J4 B2_SEL, J5 B1_SEL, Q1 BC547, SW1 P1_SEL, SW2 P2_SEL, U1 74HCT4053, U2 74HCT4053, U3 NE555, U4 NE555

Commit message: Layout done. PCB ready for manufacturing.
Parts:
- C1, C2, C3, C4: footprint Capacitors_THT:C_Disc_D4.7mm_W2.5mm_P5.00mm -> Capacitor_SMD:C_0603_1608Metric; symbol C_Small -> C64-Joystick-Switcher-rescue:C_Small; JLCPCB (none) -> C14663
- C5: footprint Capacitors_THT:CP_Radial_D5.0mm_P2.50mm -> Capacitor_Tantalum_SMD:CP_EIA-3216-18_Kemet-A; symbol CP_Small -> C64-Joystick-Switcher-rescue:CP_Small; JLCPCB (none) -> C7171
- D1, D2: footprint LEDs:LED_D5.0mm -> LED_SMD:LED_0603_1608Metric; symbol LED_Small -> C64-Joystick-Switcher-rescue:LED_Small; JLCPCB (none) -> C2286
- J1: symbol Atari_Joystick_Passive -> C64-Joystick-Switcher-rescue:Atari_Joystick_Passive
- J2, J3: symbol Atari_Joystick -> C64-Joystick-Switcher-rescue:Atari_Joystick
- J4, J5: symbol Conn_02x03_Odd_Even -> C64-Joystick-Switcher-rescue:Conn_02x03_Odd_Even
- JP1: symbol Jumper_NO_Small -> C64-Joystick-Switcher-rescue:Jumper_NO_Small
- JP2: symbol Jumper_NC_Dual -> C64-Joystick-Switcher-rescue:Jumper_NC_Dual
- Q1: value BC547 -> BC847; footprint TO_SOT_Packages_THT:TO-92_Inline_Wide -> Package_TO_SOT_SMD:SOT-23; symbol BC547 -> Transistor_BJT:BC847; JLCPCB (none) -> C57668
- R1, R2: footprint Resistors_THT:R_Axial_DIN0207_L6.3mm_D2.5mm_P10.16mm_Horizontal -> Resistor_SMD:R_0603_1608Metric; symbol R -> C64-Joystick-Switcher-rescue:R; JLCPCB (none) -> C25804
- R3, R4: footprint Resistors_THT:R_Axial_DIN0207_L6.3mm_D2.5mm_P10.16mm_Horizontal -> Resistor_SMD:R_0603_1608Metric; symbol R -> C64-Joystick-Switcher-rescue:R; JLCPCB (none) -> C22962
- R5, R7: footprint Resistors_THT:R_Axial_DIN0207_L6.3mm_D2.5mm_P10.16mm_Horizontal -> Resistor_SMD:R_0603_1608Metric; symbol R -> C64-Joystick-Switcher-rescue:R; JLCPCB (none) -> C4190
- R6: footprint Resistors_THT:R_Axial_DIN0207_L6.3mm_D2.5mm_P10.16mm_Horizontal -> Resistor_SMD:R_0603_1608Metric; symbol R -> C64-Joystick-Switcher-rescue:R; JLCPCB (none) -> C25803
- R8: renamed from R9; footprint Resistors_THT:R_Axial_DIN0207_L6.3mm_D2.5mm_P10.16mm_Horizontal -> Resistor_SMD:R_0603_1608Metric; symbol R -> C64-Joystick-Switcher-rescue:R; JLCPCB (none) -> C25804
- RV1: footprint Potentiometers:Potentiometer_Triwood_RM-065 -> Potentiometer_THT:Potentiometer_Piher_PT-6-V_Vertical; symbol POT -> C64-Joystick-Switcher-rescue:POT
- SW1, SW2: footprint Buttons_Switches_THT:SW_PUSH_6mm -> Button_Switch_THT:SW_Tactile_SPST_Angled_PTS645Vx58-2LFS; symbol SW_Push -> C64-Joystick-Switcher-rescue:SW_Push
- U1, U2: value 74HCT4053 -> 74HCT4053D; footprint Housings_DIP:DIP-16_W7.62mm_Socket -> Package_SO:SO-16_3.9x9.9mm_P1.27mm; symbol 74HCT4053 -> C64-Joystick-Switcher-rescue:74HCT4053; JLCPCB (none) -> C5996
- U3, U4: value NE555 -> TLC555CDR; footprint Housings_DIP:DIP-8_W7.62mm_Socket -> Package_SO:SO-8_3.9x4.9mm_P1.27mm; symbol NE555 -> C64-Joystick-Switcher-rescue:NE555; JLCPCB (none) -> C6986
Connections:
- wire segments 155 -> 192
